Commit message: Gripper and camera

File: UR5eWithRobotiqHandE/ur_robotiq_description/urdf/ur5e_with_robotiq_hande.xacro (robot description, xacro)
@@ -29,5 +29,5 @@
     <parent link="world"/>
     <child link="table"/>
-    <origin xyz="0 0 -0.15" rpy="0 0 0"/>
+    <origin xyz="0 0 -0.0" rpy="0 0 0"/>
   </joint>
   <!-- Define the gripper's tool center point (TCP) position and orientation WRT the flange connector -->
